Commit message: add base link
Signed-off-by: Masaya Kataoka <ms.kataoka@gmail.com>

File: urdf/miniv.urdf.xacro (robot description, xacro)
@@ -1,3 +1,7 @@
 <?xml version="1.0"?>
 <robot xmlns:xacro="http://ros.org/wiki/xacro" name="mini-v">
+  <link name="base_link"/>
+  <xacro:include filename="$(find miniv_description)/urdf/azimuth_thruster.xacro"/>
+  <xacro:azimuth_thruster prefix="right" position="-1.0 -0.25 -0.1" orientation="0 0 0"/>
+  <xacro:azimuth_thruster prefix="left" position="-1.0 0.25 -0.1" orientation="0 0 0"/>
 </robot>

Commit message: update rviz
Signed-off-by: Masaya Kataoka <ms.kataoka@gmail.com>

File: urdf/miniv.urdf.xacro (robot description, xacro)
@@ -1,5 +1,12 @@
 <?xml version="1.0"?>
 <robot xmlns:xacro="http://ros.org/wiki/xacro" name="mini-v">
-  <link name="base_link"/>
+  <link name="base_link">
+    <visual>
+      <origin xyz="0 -0.4 0" rpy="1.570795 0 1.570795"/>
+      <geometry>
+        <mesh filename="package://miniv_description/model/A_MINI_POLARIS_main.stl" scale="0.001 0.001 0.001"/>
+      </geometry>
+    </visual>
+  </link>
   <xacro:include filename="$(find miniv_description)/urdf/azimuth_thruster.xacro"/>
   <xacro:azimuth_thruster prefix="right" position="-1.0 -0.25 -0.1" orientation="0 0 0"/>
