Commit message: update stl
Signed-off-by: Masaya Kataoka <ms.kataoka@gmail.com>

File: urdf/azimuth_thruster.xacro (robot description, xacro)
@@ -3,4 +3,10 @@
   <xacro:macro name="azimuth_thruster" params="prefix position:='0 0 0' orientation:='0 0 0'">
   <link name="${prefix}_azimuth_link">
+    <visual>
+      <origin xyz="-0.025 0.0 -0.05" rpy="1.570795 0 1.570795"/>
+      <geometry>
+        <mesh filename="package://miniv_description/model/A_MINI_POLARIS_thruster.stl" scale="0.001 0.001 0.001"/>
+      </geometry>
+    </visual>
   </link>
   <joint name ="${prefix}_azimuth_link" type="fixed">

File: urdf/miniv.urdf.xacro (robot description, xacro)
@@ -1,14 +1,19 @@
 <?xml version="1.0"?>
-<robot xmlns:xacro="http://ros.org/wiki/xacro" name="mini-v">
+<robot
+    name="mini-v"
+    xmlns:xacro="http://ros.org/wiki/xacro"
+    xmlns:sensor="http://playerstage.sourceforge.net/gazebo/xmlschema/#sensor"
+    xmlns:controller="http://playerstage.sourceforge.net/gazebo/xmlschema/#controller"
+    xmlns:interface="http://playerstage.sourceforge.net/gazebo/xmlschema/#interface">>
   <link name="base_link">
     <visual>
-      <origin xyz="0 -0.4 0" rpy="1.570795 0 1.570795"/>
+      <origin xyz="0 0 0" rpy="0 0 0"/>
       <geometry>
-        <mesh filename="package://miniv_description/model/A_MINI_POLARIS_main.stl" scale="0.001 0.001 0.001"/>
+        <mesh filename="package://miniv_description/model/A_MINI_POLARIS_main_r1.stl" scale="1 1 1"/>
       </geometry>
     </visual>
   </link>
   <xacro:include filename="$(find miniv_description)/urdf/azimuth_thruster.xacro"/>
-  <xacro:azimuth_thruster prefix="right" position="-1.0 -0.25 -0.1" orientation="0 0 0"/>
-  <xacro:azimuth_thruster prefix="left" position="-1.0 0.25 -0.1" orientation="0 0 0"/>
+  <xacro:azimuth_thruster prefix="right" position="-0.51 -0.17 -0.17" orientation="0 0 0"/>
+  <xacro:azimuth_thruster prefix="left" position="-0.51 0.17 -0.17" orientation="0 0 0"/>
 </robot>

Commit message: update rviz and controller
Signed-off-by: Masaya Kataoka <ms.kataoka@gmail.com>

File: urdf/azimuth_thruster.xacro (robot description, xacro)
@@ -1,4 +1,4 @@
 <?xml version="1.0"?>
-<robot xmlns:xacro="http://ros.org/wiki/xacro" name="wam-v-batteries">
+<robot xmlns:xacro="http://ros.org/wiki/xacro" name="azimuth_thruster">
   <xacro:macro name="azimuth_thruster" params="prefix position:='0 0 0' orientation:='0 0 0'">
   <link name="${prefix}_azimuth_link">
@@ -10,5 +10,5 @@
     </visual>
   </link>
-  <joint name ="${prefix}_azimuth_link" type="fixed">
+  <joint name ="${prefix}_azimuth_joint" type="fixed">
     <origin xyz="${position}" rpy="${orientation}"/>
     <parent link="base_link"/>

File: urdf/miniv.urdf.xacro (robot description, xacro)
@@ -5,5 +5,5 @@
     xmlns:sensor="http://playerstage.sourceforge.net/gazebo/xmlschema/#sensor"
     xmlns:controller="http://playerstage.sourceforge.net/gazebo/xmlschema/#controller"
-    xmlns:interface="http://playerstage.sourceforge.net/gazebo/xmlschema/#interface">>
+    xmlns:interface="http://playerstage.sourceforge.net/gazebo/xmlschema/#interface">
   <link name="base_link">
     <visual>
@@ -14,14 +14,5 @@
     </visual>
   </link>
-  <ros2_control name="miniv_control" type="system">
-    <hardware>
-      <plugin>miniv_control/MiniVHardware</plugin>
-      <param name="thruster_ip_address">192.168.0.25</param>
-      <param name="port">8000</param>
-      <param name="timeout_seconds">10.0</param>
-    </hardware>
-  </ros2_control>
-  <xacro:include filename="$(find miniv_description)/urdf/azimuth_thruster.xacro"/>
-  <xacro:azimuth_thruster prefix="right" position="-0.51 -0.17 -0.17" orientation="0 0 0"/>
-  <xacro:azimuth_thruster prefix="left" position="-0.51 0.17 -0.17" orientation="0 0 0"/>
+  <xacro:include filename="$(find miniv_description)/urdf/thruster.xacro"/>
+  <xacro:thruster control_azimuth="true"/>
 </robot>
