Commit message: comment out error section
Signed-off-by: Masaya Kataoka <ms.kataoka@gmail.com>

File: urdf/miniv.ros2_control.xacro (robot description, xacro)
@@ -28,13 +28,14 @@
     </ros2_control>
   </xacro:macro>
-  <xacro:macro name="main_thruster_control" params="left_joint right_joint">
+  <xacro:macro name="main_thruster_control" params="ip_address port">
     <ros2_control name="main_thruster_control" type="system">
+<!--
       <hardware>
         <plugin>miniv_control/MiniVHardware</plugin>
-        <param name="thruster_ip_address">${thruster_ip_address}</param>
-        <param name="port">${thruster_port}</param>
+        <param name="ip_address">${ip_address}</param>
+        <param name="port">${port}</param>
         <param name="timeout_seconds">10.0</param>
-        <param name="enable_azimuth">${control_azimuth}</param>
       </hardware>
+-->
     </ros2_control>
   </xacro:macro>

File: urdf/thruster.xacro (robot description, xacro)
@@ -5,10 +5,11 @@
   xmlns:controller="http://playerstage.sourceforge.net/gazebo/xmlschema/#controller"
   xmlns:interface="http://playerstage.sourceforge.net/gazebo/xmlschema/#interface">
-  <xacro:include filename="$(find miniv_description)/urdf/miniv.ros2_control.xacro"/>
   <xacro:macro name="thruster" params="control_azimuth thruster_ip_address='192.168.0.25' thruster_port=12345">
     <xacro:include filename="$(find miniv_description)/urdf/azimuth_thruster.xacro"/>
     <xacro:azimuth_thruster prefix="right" position="-0.51 -0.17 -0.17" orientation="0 0 0"/>
     <xacro:azimuth_thruster prefix="left" position="-0.51 0.17 -0.17" orientation="0 0 0"/>
+    <xacro:include filename="$(find miniv_description)/urdf/miniv.ros2_control.xacro"/>
     <xacro:azimuth_thruster_control left_joint="left_azimuth_joint" right_joint="right_azimuth_joint"/>
+    <xacro:main_thruster_control ip_address="${thruster_ip_address}" port="${thruster_port}"/>
   </xacro:macro>
 </robot>

Commit message: update thruster macro
Signed-off-by: Masaya Kataoka <ms.kataoka@gmail.com>

File: urdf/miniv.ros2_control.xacro (robot description, xacro)
@@ -28,7 +28,6 @@
     </ros2_control>
   </xacro:macro>
-  <xacro:macro name="main_thruster_control" params="ip_address port">
+  <xacro:macro name="main_thruster_control" params="ip_address port left_thruster_joint right_thruster_joint">
     <ros2_control name="main_thruster_control" type="system">
-<!--
       <hardware>
         <plugin>miniv_control/MiniVHardware</plugin>
@@ -36,6 +35,7 @@
         <param name="port">${port}</param>
         <param name="timeout_seconds">10.0</param>
+        <param name="left_thruster_joint">${left_thruster_joint}</param>
+        <param name="right_thruster_joint">${right_thruster_joint}</param>
       </hardware>
--->
     </ros2_control>
   </xacro:macro>

File: urdf/thruster.xacro (robot description, xacro)
@@ -9,7 +9,14 @@
     <xacro:azimuth_thruster prefix="right" position="-0.51 -0.17 -0.17" orientation="0 0 0"/>
     <xacro:azimuth_thruster prefix="left" position="-0.51 0.17 -0.17" orientation="0 0 0"/>
+    <xacro:include filename="$(find miniv_description)/urdf/main_thruster.xacro"/>
+    <xacro:main_thruster prefix="right" position="0.0 0.0 -0.05" orientation="0 0 3.14159265359"/>
+    <xacro:main_thruster prefix="left" position="0.0 0.0 -0.05" orientation="0 0 3.14159265359"/>
     <xacro:include filename="$(find miniv_description)/urdf/miniv.ros2_control.xacro"/>
     <xacro:azimuth_thruster_control left_joint="left_azimuth_joint" right_joint="right_azimuth_joint"/>
-    <xacro:main_thruster_control ip_address="${thruster_ip_address}" port="${thruster_port}"/>
+    <xacro:main_thruster_control
+      ip_address="${thruster_ip_address}"
+      port="${thruster_port}"
+      left_thruster_joint="left_thruster_joint"
+      right_thruster_joint="right_thruster_joint"/>
   </xacro:macro>
 </robot>

Commit message: add enable_dummy parameter
Signed-off-by: Masaya Kataoka <ms.kataoka@gmail.com>

File: urdf/miniv.ros2_control.xacro (robot description, xacro)
@@ -1,4 +1,4 @@
 <robot xmlns:xacro="http://ros.org/wiki/xacro" name="azimuth_thruster">
-  <xacro:macro name="azimuth_thruster_control" params="left_joint right_joint">
+  <xacro:macro name="azimuth_thruster_control" params="left_joint right_joint enable_dummy">
     <ros2_control name="azimuth_thruster_control" type="system">
       <hardware>
@@ -6,5 +6,5 @@
         <param name="port_name">/dev/ttyUSB0</param>
         <param name="baudrate">9600</param>
-        <param name="enable_dummy">false</param>
+        <param name="enable_dummy">${enable_dummy}</param>
       </hardware>
       <joint name="${left_joint}">
@@ -22,5 +22,5 @@
     </ros2_control>
   </xacro:macro>
-  <xacro:macro name="main_thruster_control" params="ip_address port left_thruster_joint right_thruster_joint">
+  <xacro:macro name="main_thruster_control" params="ip_address port left_thruster_joint right_thruster_joint enable_dummy">
     <ros2_control name="main_thruster_control" type="system">
       <hardware>
@@ -31,4 +31,5 @@
         <param name="left_thruster_joint">${left_thruster_joint}</param>
         <param name="right_thruster_joint">${right_thruster_joint}</param>
+        <param name="enable_dummy">${enable_dummy}</param>
       </hardware>
     </ros2_control>

File: urdf/miniv_robot.urdf.xacro (robot description, xacro)
@@ -15,4 +15,4 @@
   </link>
   <xacro:include filename="$(find miniv_description)/urdf/thruster.xacro"/>
-  <xacro:thruster control_azimuth="true"/>
+  <xacro:thruster enable_dummy="false"/>
 </robot>

File: urdf/thruster.xacro (robot description, xacro)
@@ -5,5 +5,5 @@
   xmlns:controller="http://playerstage.sourceforge.net/gazebo/xmlschema/#controller"
   xmlns:interface="http://playerstage.sourceforge.net/gazebo/xmlschema/#interface">
-  <xacro:macro name="thruster" params="control_azimuth thruster_ip_address='192.168.0.25' thruster_port=12345">
+  <xacro:macro name="thruster" params="enable_dummy thruster_ip_address='192.168.0.25' thruster_port=12345">
     <xacro:include filename="$(find miniv_description)/urdf/azimuth_thruster.xacro"/>
     <xacro:azimuth_thruster prefix="right" position="-0.51 -0.17 -0.17" orientation="0 0 0"/>
@@ -13,6 +13,10 @@
     <xacro:main_thruster prefix="left" position="0.0 0.0 -0.05" orientation="0 0 3.14159265359"/>
     <xacro:include filename="$(find miniv_description)/urdf/miniv.ros2_control.xacro"/>
-    <xacro:azimuth_thruster_control left_joint="left_azimuth_joint" right_joint="right_azimuth_joint"/>
+    <xacro:azimuth_thruster_control
+      left_joint="left_azimuth_joint"
+      right_joint="right_azimuth_joint"
+      enable_dummy="${enable_dummy}"/>
     <xacro:main_thruster_control
+      enable_dummy="${enable_dummy}"
       ip_address="${thruster_ip_address}"
       port="${thruster_port}"

Commit message: update xacro
Signed-off-by: Masaya Kataoka <ms.kataoka@gmail.com>

File: urdf/miniv.ros2_control.xacro (robot description, xacro)
@@ -1,3 +1,14 @@
 <robot xmlns:xacro="http://ros.org/wiki/xacro" name="azimuth_thruster">
+  <xacro:macro name="realsense_hardware_interface">
+    <ros2_control name="t265_control" type="sensor">
+      <hardware>
+        <plugin>realsense_hardware_interface/T265HardwareInterface</plugin>
+        <param name="retrive_image">false</param>
+        <param name="left_image_key">t265_left_fisheye</param>
+        <param name="right_image_key">t265_right_fisheye</param>
+        <param name="serial">109422110714</param>
+      </hardware>
+    </ros2_control>
+  </xacro:macro>
   <xacro:macro name="azimuth_thruster_control" params="left_joint right_joint enable_dummy">
     <ros2_control name="azimuth_thruster_control" type="system">

Commit message: add hardware interface to the xacro file
Signed-off-by: Masaya Kataoka <ms.kataoka@gmail.com>

File: urdf/miniv.ros2_control.xacro (robot description, xacro)
@@ -1,14 +1,3 @@
 <robot xmlns:xacro="http://ros.org/wiki/xacro" name="azimuth_thruster">
-  <xacro:macro name="realsense_hardware_interface">
-    <ros2_control name="t265_control" type="sensor">
-      <hardware>
-        <plugin>realsense_hardware_interface/T265HardwareInterface</plugin>
-        <param name="retrive_image">false</param>
-        <param name="left_image_key">t265_left_fisheye</param>
-        <param name="right_image_key">t265_right_fisheye</param>
-        <param name="serial">109422110714</param>
-      </hardware>
-    </ros2_control>
-  </xacro:macro>
   <xacro:macro name="azimuth_thruster_control" params="left_joint right_joint enable_dummy">
     <ros2_control name="azimuth_thruster_control" type="system">

File: urdf/miniv_robot.urdf.xacro (robot description, xacro)
@@ -21,4 +21,13 @@
     <child link="t265_link"/>
   </joint>
+  <ros2_control name="t265_control" type="sensor">
+    <hardware>
+      <plugin>realsense_hardware_interface/T265HardwareInterface</plugin>
+      <param name="retrive_image">false</param>
+      <param name="left_image_key">t265_left_fisheye</param>
+      <param name="right_image_key">t265_right_fisheye</param>
+      <param name="serial">109422110714</param>
+    </hardware>
+  </ros2_control>
   <xacro:include filename="$(find miniv_description)/urdf/thruster.xacro"/>
   <xacro:thruster enable_dummy="false"/>
