Commit message: add t265_link
Signed-off-by: Masaya Kataoka <ms.kataoka@gmail.com>

File: urdf/miniv_robot.urdf.xacro (robot description, xacro)
@@ -14,4 +14,11 @@
     </visual>
   </link>
+  <link name="t265_link">
+  </link>
+  <joint name ="t265_joint" type="fixed">
+    <origin xyz="0.4 0 0" rpy="0 0 0"/>
+    <parent link="base_link"/>
+    <child link="t265_link"/>
+  </joint>
   <xacro:include filename="$(find miniv_description)/urdf/thruster.xacro"/>
   <xacro:thruster enable_dummy="false"/>

Commit message: modify xacro
Signed-off-by: Masaya Kataoka <ms.kataoka@gmail.com>

File: urdf/miniv_robot.urdf.xacro (robot description, xacro)
@@ -29,4 +29,6 @@
       <param name="serial">109422110714</param>
     </hardware>
+    <joint name="t265_link">
+    </joint>
   </ros2_control>
   <xacro:include filename="$(find miniv_description)/urdf/thruster.xacro"/>

Commit message: modify realsense position
Signed-off-by: Masaya Kataoka <ms.kataoka@gmail.com>

File: urdf/miniv_robot.urdf.xacro (robot description, xacro)
@@ -17,5 +17,5 @@
   </link>
   <joint name ="t265_joint" type="fixed">
-    <origin xyz="0.4 0 0" rpy="0 0 0"/>
+    <origin xyz="0.3 0 0.15" rpy="0 0 0"/>
     <parent link="base_link"/>
     <child link="t265_link"/>
